File: kicad/eepromgramer.kicad_sch (KiCad schematic)
At the start: 35 parts, among them J1 arduino header, J2 data header, J3 address header, J4 eeprom generic connector, SW1 SW_DIP_x10, SW2 SW_DIP_x04, U1 74AHC595, U2 74AHC595, U3 74AHC595, U4 74AHC595, U5 74HC165

Commit message: updates
Parts:
- removed SW2: SW_DIP_x04, symbol Switch:SW_DIP_x04
- added D?: 1N4148, Diode_THT:D_DO-35_SOD27_P7.62mm_Horizontal, symbol Diode:1N4148
- added J6: external vpp2 14V, symbol Connector:Conn_01x02_Female
- added SW2: SW_DIP_x10, symbol Switch:SW_DIP_x10
- D4: renamed from D?; value (none) -> GREEN
- D5: renamed from D?; value (none) -> RED
- J5: value (none) -> external vpp 12.75V
- R8: renamed from R2; value (none) -> 4k7
- gave numbers to parts that had none: 7
- renumbered D3 to D1
Connections:
- net HSER1 is gone; now on net SER1: U1.14 (SER)
- net A14: now also SW2.17
- net A15: now also SW2.18
- net A18: now also SW2.12, SW2.19; no longer J4.5 (Pin_5)
- net EEWE: now also SW2.11; no longer J4.35 (Pin_35)
- net GND: now also D?.2 (A)
- net T06: now also J4.35 (Pin_35), SW2.10, SW2.9; no longer J4.7 (Pin_7)
- net +12V renamed VPP
- net VPP: now also SW2.16, SW2.20
- net +5V renamed VCC
- net VCC: now also SW2.14; no longer J4.36 (Pin_36)
- net LSER1: no longer names the net of U1.9 (QH'), U2.14 (SER)
- new net: D?.1 (K), J6.1 (Pin_1)
- new net NCC: SW2.13
- new net T07: J4.36 (Pin_36), SW2.7, SW2.8
- new net T08: J4.7 (Pin_7), SW2.3, SW2.4, SW2.5, SW2.6
- new net T09: J4.5 (Pin_5), SW2.1, SW2.2
- new net VPP2: J6.2 (Pin_2), SW2.15
Other:
- note added: "VCC must be 5.0V +/- 0.5V VPP must be 12.75 V +/- 0.25 V VPP2 must be 12V to program or 14V to erase J1 if arduino in other pcb J2 and J3 if eeprom J4 in other pcb"
- note added: "dip switch 01 and 02 for eeproms: AT28C16, (01 ON: S6, S8, S9), (02 ON: S3) AT28C64, (01 ON: S2, S4, S7, S9), (02 ON: S3) AT28C256, (01 ON: S2, S4, S7, S9), (02 ON: S4)** SST39SF040, (01 ON: S1, S3, S5, S7, S9), (02 ON: S3) M27C512, (01 ON: S2, S3, S5, S7, S10), (02 ON: S3) A27E257 to review AT24CXXX ALL OFF."
- note removed: "Address switch, HSER1 use higher address as serial input LSER1 use lower address as serial input"
- note removed: "VPP must be 12.75 V +/- 0.25 V J1 if arduino in other pcb J2 and J3 if eeprom J4 in other pcb I2C and SPI share same wires"
- note removed: "dip switch 01 and 02 for eeproms: AT28C16, (01 ON: S6, S8, S9), (02 ON: S3) AT28C64, (01 ON: S2, S4, S7, S9), (02 ON: S3) AT28C256, (01 ON: S2, S4, S7, S9), (02 ON: S4)** SST39SF040, (01 ON: S1, S3, S5, S7, S9), (02 ON: S3) M27C512, (01 ON: S2, S3, S5, S7, S10), (02 ON: S3) AT24CXXX ALL OFF."
- moved on the sheet: D2, D3, D4, D5, J5, R1, R2, R3, R4, R5, R6, R8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
