File: kicad/eeprogram.detail.pins.kicad_sch (KiCad schematic)
At the start: 3 parts, among them J3 Conn_02x20_Top_Bottom

Commit message: updates
Parts:
- removed SW?: SW_DIP_x12, symbol Switch:SW_DIP_x12
- added J1: I2C, symbol Connector_Generic:Conn_02x04_Counter_Clockwise
- added J2: SPI, symbol Connector_Generic:Conn_02x04_Counter_Clockwise
Connections:
- net A10: now also J3.34 (Pin_34); no longer J3.28 (Pin_28)
- net A11: now also J3.32 (Pin_32); no longer J3.26 (Pin_26)
- net A12: now also J3.8 (Pin_8); no longer J3.2 (Pin_2)
- net A13: now also J3.29 (Pin_29); no longer J3.23 (Pin_23)
- net A14: now also J3.7 (Pin_7); no longer J3.1 (Pin_1)
- net A3: now also J3.13 (Pin_13); no longer J3.7 (Pin_7)
- net A4: now also J3.12 (Pin_12); no longer J3.6 (Pin_6)
- net A5: now also J3.11 (Pin_11); no longer J3.5 (Pin_5)
- net A6: now also J3.10 (Pin_10); no longer J3.4 (Pin_4)
- net A7: now also J3.9 (Pin_9); no longer J3.3 (Pin_3)
- net A8: now also J3.30 (Pin_30); no longer J3.24 (Pin_24)
- net A9: now also J3.31 (Pin_31); no longer J3.25 (Pin_25)
- net D0: now also J3.17 (Pin_17); no longer J3.11 (Pin_11)
- net D1: now also J3.18 (Pin_18); no longer J3.12 (Pin_12)
- net D2: now also J3.19 (Pin_19); no longer J3.13 (Pin_13)
- net D3: now also J3.40 (Pin_40); no longer J3.34 (Pin_34)
- net D4: now also J3.39 (Pin_39); no longer J3.33 (Pin_33)
- net D5: now also J3.38 (Pin_38); no longer J3.32 (Pin_32)
- net D6: now also J3.37 (Pin_37); no longer J3.31 (Pin_31)
- net D7: now also J3.36 (Pin_36); no longer J3.30 (Pin_30)
- net GND: now also J3.15 (Pin_15), J3.16 (Pin_16), J1.1 (Pin_1), J1.2 (Pin_2), J1.3 (Pin_3), J1.4 (Pin_4), J2.4 (Pin_4)
- net MOSI: now also J2.6 (Pin_6); no longer J3.40 (Pin_40)
- net SCK: now also J2.7 (Pin_7); no longer J3.39 (Pin_39)
- net VCC: now also J3.27 (Pin_27), J1.8 (Pin_8), J2.8 (Pin_8); no longer J3.21 (Pin_21), J3.37 (Pin_37)
- net WP: now also J1.5 (Pin_5); no longer J3.38 (Pin_38)
- net /CE: now also J3.35 (Pin_35); no longer J3.29 (Pin_29)
- net /OE: now also J3.33 (Pin_33); no longer J3.27 (Pin_27)
- net /WE: now also J3.28 (Pin_28); no longer J3.22 (Pin_22)
- removed net A0: J3.10 (Pin_10), J3.17 (Pin_17)
- removed net A1: J3.18 (Pin_18), J3.9 (Pin_9)
- removed net A2: J3.19 (Pin_19), J3.8 (Pin_8)
- new net MISO: J2.5 (Pin_5)
- new net SCL: J1.6 (Pin_6)
- new net SDA: J1.7 (Pin_7)
- new net /CS: J2.3 (Pin_3)
- new net /HOLD: J2.2 (Pin_2)
- new net /WP: J2.1 (Pin_1)
- no-connect marks 4 -> 0
Other:
- note added: "adapted from https://tomnisbet.github.io/TommyPROM/docs/hardware, include I2C and SPI use agsb@"
- moved on the sheet: J3
