File: kicad/eeprogram.chips.kicad_sch (KiCad schematic)
At the start: 12 parts, among them J5 Conn_01x04_Female, U2 28C256, U3 74HC595, U4 74HC595

Commit message: updates
Parts:
- added C5, C6: C, symbol Device:C
- added U1: 25LCxxx, symbol Memory_EEPROM:25LCxxx
- added U5: 24LC256, symbol Memory_EEPROM:24LC256
Connections:
- net A15: now also U3.12 (RCLK), U4.12 (RCLK), U1.1 (~{CS})
- net A16: now also U1.5 (MOSI)
- net A17: now also U1.2 (MISO)
- net GND: now also A1.29 (GND), A1.4 (GND), C5.2, C6.2, U1.4 (GND), U5.1 (A0), U5.2 (A1), U5.3 (A2), U5.4 (GND), U5.7 (WP)
- net VCC: now also C5.1, C6.1, U1.3 (~{WP}), U1.8 (VCC), U5.8 (VCC)
- net at A1.12 (D9), U2.19 (D7): now also U1.7 (~{HOLD})
- net at A1.22 (A3): now also U3.11 (SRCLK); no longer U4.11 (SRCLK)
- net SCL: now reaches A1.24 (A5), U3.14 (SER), U4.14 (SER)
- net SCL: now also U5.6 (SCL)
- net SDA: now reaches A1.23 (A4)
- net SDA: now also U4.11 (SRCLK), U5.5 (SDA); no longer U3.11 (SRCLK)
- new net A18: A1.16 (D13), U1.6 (SCK)
- no-connect marks 11 -> 12
Other:
- note added: "adapted from https://tomnisbet.github.io/TommyPROM/docs/hardware, include I2C and SPI use agsb@"
- moved on the sheet: A1, C1, J5, R5, R6

Commit message: update schematics
Parts:
- added D1, D11, D12, D13, D14, D15, D16, D17, D18, D2, D3, D4, D5, D6, D7, D8: LED, LED_THT:LED_D5.0mm_Clear, symbol Device:LED
- added R1, R11, R12, R13, R14, R15, R16, R17, R18, R2, R3, R4, R5, R6, R7, R8: R_US, Resistor_THT:R_Box_L8.4mm_W2.5mm_P5.08mm, symbol Device:R_US
- renumbered R4 to R21, R5 to R22, R6 to R23
Connections:
- net +3.3V: now also U1.3 (~{WP}), U1.8 (VCC), U5.8 (VCC)
- net GND: now also D1.1 (K), D11.1 (K), D12.1 (K), D13.1 (K), D14.1 (K), D15.1 (K), D16.1 (K), D17.1 (K), D18.1 (K), D2.1 (K), D3.1 (K), D4.1 (K), D5.1 (K), D6.1 (K), D7.1 (K), D8.1 (K)
- net VCC: no longer A1.27 (+5V), U1.3 (~{WP}), U1.8 (VCC), U2.28 (VCC), U3.10 (~{SRCLR}), U3.16 (VCC), U4.10 (~{SRCLR}), U4.16 (VCC), U5.8 (VCC)
- net at U2.1 (A14), U4.6 (QG): now also R7.1
- net at U2.10 (A0), U3.15 (QA): now also R11.1
- net at U2.2 (A12), U4.4 (QE): now also R5.1
- net at U2.21 (A10), U4.2 (QC): now also R3.1
- net at U2.23 (A11), U4.3 (QD): now also R4.1
- net at U2.24 (A9), U4.1 (QB): now also R2.1
- net at U2.25 (A8), U4.15 (QA): now also R1.1
- net at U2.26 (A13), U4.5 (QF): now also R6.1
- net at U2.3 (A7), U3.7 (QH): now also R18.1
- net at U2.4 (A6), U3.6 (QG): now also R17.1
- net at U2.5 (A5), U3.5 (QF): now also R16.1
- net at U2.6 (A4), U3.4 (QE): now also R15.1
- net at U2.7 (A3), U3.3 (QD): now also R14.1
- net at U2.8 (A2), U3.2 (QC): now also R13.1
- net at U2.9 (A1), U3.1 (QB): now also R12.1
- net at U4.7 (QH): now also R8.1
- new net: D2.2 (A), R2.2
- new net: D17.2 (A), R17.2
- new net: D8.2 (A), R8.2
- new net: D18.2 (A), R18.2
- new net: D3.2 (A), R3.2
- new net: D15.2 (A), R15.2
- new net: D14.2 (A), R14.2
- new net: D6.2 (A), R6.2
- new net: D13.2 (A), R13.2
- new net: D5.2 (A), R5.2
- new net: D11.2 (A), R11.2
- new net: D12.2 (A), R12.2
- new net: D4.2 (A), R4.2
- new net: D7.2 (A), R7.2
- new net: D1.2 (A), R1.2
- new net: D16.2 (A), R16.2
- new net 5V0: A1.27 (+5V), U2.28 (VCC), U3.10 (~{SRCLR}), U3.16 (VCC), U4.10 (~{SRCLR}), U4.16 (VCC)
- no-connect marks 12 -> 11
Other:
- moved on the sheet: C1, C2, C3, C4, C5, C6, U3, U4

Commit message: update wire list
Connections:
- net A15: now also R8.1, U4.7 (QH); no longer A1.13 (D10), U1.1 (~{CS}), U3.12 (RCLK), U4.12 (RCLK)
- net A16: now also A1.13 (D10), U1.1 (~{CS}); no longer A1.14 (D11), U1.5 (MOSI)
- net A17: now also A1.14 (D11), U1.5 (MOSI); no longer A1.15 (D12), U1.2 (MISO)
- net A18: now also A1.15 (D12), U1.2 (MISO); no longer A1.16 (D13), U1.6 (SCK)
- new net SCK: A1.16 (D13), U1.6 (SCK), U3.12 (RCLK), U4.12 (RCLK)
- no-connect marks 11 -> 10
