File: kicad/eeprogrammer.kicad_sch (KiCad schematic)
At the start: 0 parts

Commit message: update wire list
Changed lines of the file:
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@@
 	)
 	(sheet
-		(at 86.36 25.4)
+		(at 111.76 40.64)
 		(size 43.815 19.685)
 		(exclude_from_sim no)
@@
 		)
 		(property "Sheetname" "pins wires"
-			(at 86.36 24.6884 0)
+			(at 111.76 39.9284 0)
 			(effects
 				(font
@@
 		)
 		(property "Sheetfile" "eeprogram.detail.pins.kicad_sch"
-			(at 86.36 45.6696 0)
+			(at 111.76 60.9096 0)
 			(effects
 				(font
@@
 	)
 	(sheet
-		(at 27.305 26.035)
+		(at 52.705 41.275)
 		(size 43.815 19.685)
 		(exclude_from_sim no)
@@
 		)
 		(property "Sheetname" "chips"
-			(at 27.305 25.3234 0)
+			(at 52.705 40.5634 0)
 			(effects
 				(font
@@
 		)
 		(property "Sheetfile" "eeprogram.chips.kicad_sch"
-			(at 27.305 46.3046 0)
+			(at 52.705 61.5446 0)
 			(effects
 				(font
